Commit message: update

File: jackal_description/urdf/jackal.urdf.xacro (robot description, xacro)
@@ -243,3 +243,9 @@
   <!-- Optional for Clearpath internal softwares -->
   <xacro:include filename="$(optenv CPR_URDF_EXTRAS empty.urdf)" />
+  <xacro:include filename="$(find servo_mapping)/urdf/qr1.urdf.xacro"/>
+  <joint name="qrGlue" type="fixed">
+    <parent link="rear_mount"/>
+    <child link="qrcode"/>
+    <origin xyz="0 0 0"/>
+  </joint>
 </robot>

Commit message: update

File: jackal_description/urdf/jackal.urdf.xacro (robot description, xacro)
@@ -247,5 +247,5 @@
     <parent link="rear_mount"/>
     <child link="qrcode"/>
-    <origin xyz="0 0 0"/>
+    <origin xyz="0 0 0.1" rpy="0.0 1.57 0"/>
   </joint>
 </robot>

Commit message: update navigation package, added odom_gps for local localization

File: jackal_description/urdf/jackal.urdf.xacro (robot description, xacro)
@@ -239,13 +239,9 @@
        default each one to off.-->
   <xacro:include filename="$(find jackal_description)/urdf/accessories.urdf.xacro" />
-  <!-- Optional custom includes. -->
-  <xacro:include filename="$(optenv JACKAL_URDF_EXTRAS empty.urdf)" />
-  <!-- Optional for Clearpath internal softwares -->
-  <xacro:include filename="$(optenv CPR_URDF_EXTRAS empty.urdf)" />
   <xacro:include filename="$(find servo_mapping)/urdf/qr1.urdf.xacro"/>
   <joint name="qrGlue" type="fixed">
     <parent link="rear_mount"/>
     <child link="qrcode"/>
-    <origin xyz="0 0 0.1" rpy="0.0 1.57 0"/>
+    <origin xyz="0 0 0.0" rpy="0.0 0.0 0"/>
   </joint>
 </robot>

Commit message: add

File: jackal_description/urdf/jackal.urdf.xacro (robot description, xacro)
@@ -241,5 +241,5 @@
   <xacro:include filename="$(find servo_mapping)/urdf/qr1.urdf.xacro"/>
   <joint name="qrGlue" type="fixed">
-    <parent link="rear_mount"/>
+    <parent link="front_mount"/>
     <child link="qrcode"/>
     <origin xyz="0 0 0.0" rpy="0.0 0.0 0"/>

Commit message: updates

File: jackal_description/urdf/jackal.urdf.xacro (robot description, xacro)
@@ -238,10 +238,15 @@
        of these into the final description is controlled by optenv variables, which
        default each one to off.-->
-  <xacro:include filename="$(find jackal_description)/urdf/accessories.urdf.xacro" />
+  <xacro:include filename="$(find jackal_description)/urdf/custom_accessories.urdf.xacro" />
   <xacro:include filename="$(find servo_mapping)/urdf/qr1.urdf.xacro"/>
   <joint name="qrGlue" type="fixed">
     <parent link="front_mount"/>
-    <child link="qrcode"/>
-    <origin xyz="0 0 0.0" rpy="0.0 0.0 0"/>
+    <child link="qrcode10"/>
+    <origin xyz="-0.2 0 0.0" rpy="0.0 0.0 0"/>
+  </joint>
+    <joint name="qrGlue2" type="fixed">
+    <parent link="front_mount"/>
+    <child link="qrcode11"/>
+    <origin xyz="0.0 0 0.0" rpy="0.0 0.0 0"/>
   </joint>
 </robot>

Commit message: update

File: jackal_description/urdf/jackal.urdf.xacro (robot description, xacro)
@@ -240,4 +240,13 @@
   <!-- <xacro:include filename="$(find jackal_description)/urdf/custom_accessories.urdf.xacro" /> -->
   <xacro:include filename="$(find servo_mapping)/urdf/qr1.urdf.xacro"/>
+    <gazebo reference="front_fender_link">
+    <material>Gazebo/Yellow</material>
+  </gazebo>
+      <gazebo reference="rear_fender_link">
+    <material>Gazebo/Yellow</material>
+  </gazebo>
+      <gazebo reference="chassis_link">
+    <material>Gazebo/Blue</material>
+  </gazebo>
   <joint name="qrGlue" type="fixed">
     <parent link="front_mount"/>
@@ -245,8 +254,3 @@
     <origin xyz="0.0 0 0.0" rpy="0.0 0.0 0"/>
   </joint>
-    <!-- <joint name="qrGlue2" type="fixed">
-    <parent link="front_mount"/>
-    <child link="qrcode11"/>
-    <origin xyz="0.0 0 0.0" rpy="0.0 0.0 0"/>
-  </joint> -->
 </robot>

Commit message: update

File: jackal_description/urdf/jackal.urdf.xacro (robot description, xacro)
@@ -103,5 +103,6 @@
       <!-- Center of mass -->
       <origin xyz="0.012  0.002 0.067" rpy="0 0 0"/>
-      <mass value="16.523"/>
+      <!-- <mass value="16.523"/> -->
+      <mass value="30.000"/>
       <!-- Moments of inertia: ( chassis without wheels ) -->
       <inertia

Commit message: update

File: jackal_description/urdf/jackal.urdf.xacro (robot description, xacro)
@@ -239,6 +239,5 @@
        of these into the final description is controlled by optenv variables, which
        default each one to off.-->
-  <xacro:include filename="$(find jackal_description)/urdf/custom_accessories.urdf.xacro" />
-  <xacro:include filename="$(find servo_mapping)/urdf/qr1.urdf.xacro"/>
+  <!-- <xacro:include filename="$(find jackal_description)/urdf/custom_accessories.urdf.xacro" /> -->
     <gazebo reference="front_fender_link">
     <material>Gazebo/Yellow</material>
@@ -250,8 +249,3 @@
     <material>Gazebo/White</material>
   </gazebo>
-  <joint name="qrGlue" type="fixed">
-    <parent link="front_mount"/>
-    <child link="qrcode3"/>
-    <origin xyz="0.0 0 0.0" rpy="0.0 0.0 0"/>
-  </joint>
 </robot>
