Commit message: update

File: jackal_description/urdf/custom_accessories.urdf.xacro (robot description, xacro)
@@ -129,8 +129,12 @@
     </actuator>
   </transmission>
-  <!-- <gazebo reference="custom_tool_link">
-    <material>Gazebo/Yellow</material>
+  <gazebo reference="custom_tool_base_link">
+    <material>Gazebo/GreenGlow</material>
     <turnGravityOff>false</turnGravityOff>
-  </gazebo> -->
+  </gazebo>
+  <gazebo reference="custom_tool_link">
+    <material>Gazebo/GreenGlow</material>
+    <turnGravityOff>false</turnGravityOff>
+  </gazebo>
   <!-- Custom tool model. -->
 </robot>

File: jackal_description/urdf/jackal.urdf.xacro (robot description, xacro)
@@ -238,15 +238,15 @@
        of these into the final description is controlled by optenv variables, which
        default each one to off.-->
-  <xacro:include filename="$(find jackal_description)/urdf/custom_accessories.urdf.xacro" />
+  <!-- <xacro:include filename="$(find jackal_description)/urdf/custom_accessories.urdf.xacro" /> -->
   <xacro:include filename="$(find servo_mapping)/urdf/qr1.urdf.xacro"/>
   <joint name="qrGlue" type="fixed">
     <parent link="front_mount"/>
-    <child link="qrcode10"/>
-    <origin xyz="-0.2 0 0.0" rpy="0.0 0.0 0"/>
-  </joint>
-    <joint name="qrGlue2" type="fixed">
+    <child link="qrcode3"/>
+    <origin xyz="0.0 0 0.0" rpy="0.0 0.0 0"/>
+  </joint>
+    <!-- <joint name="qrGlue2" type="fixed">
     <parent link="front_mount"/>
     <child link="qrcode11"/>
     <origin xyz="0.0 0 0.0" rpy="0.0 0.0 0"/>
-  </joint>
+  </joint> -->
 </robot>

Commit message: update

File: jackal_description/urdf/custom_accessories.urdf.xacro (robot description, xacro)
@@ -54,5 +54,5 @@
   </link>
   <!-- Revolute joint. -->
-  <joint name="custom_tool_joint" type="revolute">
+  <joint name="custom_tool_joint" type="fixed">
     <parent link="custom_tool_base_link"/>
     <child link="custom_tool_link"/>
@@ -65,6 +65,6 @@
     <origin rpy="1.5707 0 -1.5707" xyz="0 0 0"/>
     <axis xyz="0 0 1"/>
-    <limit lower="-0.7853982" upper="0.7853982" effort="1000" velocity="10"/>
-    <dynamics damping="0.7"/>
+    <!-- <limit lower="-0.7853982" upper="0.7853982" effort="1000" velocity="10"/>
+    <dynamics damping="0.7"/> -->
   </joint>
   <!-- <link name="custom_tool_link">
@@ -119,5 +119,5 @@
     </inertial>
   </link>
-  <transmission name="custom_tool_trans">
+  <!-- <transmission name="custom_tool_trans">
     <type>transmission_interface/SimpleTransmission</type>
     <joint name="custom_tool_joint">
@@ -128,5 +128,5 @@
         <mechanicalReduction>1</mechanicalReduction>
     </actuator>
-  </transmission>
+  </transmission> -->
   <gazebo reference="custom_tool_base_link">
     <material>Gazebo/GreenGlow</material>

File: jackal_description/urdf/jackal.urdf.xacro (robot description, xacro)
@@ -238,5 +238,5 @@
        of these into the final description is controlled by optenv variables, which
        default each one to off.-->
-  <!-- <xacro:include filename="$(find jackal_description)/urdf/custom_accessories.urdf.xacro" /> -->
+  <xacro:include filename="$(find jackal_description)/urdf/custom_accessories.urdf.xacro" />
   <xacro:include filename="$(find servo_mapping)/urdf/qr1.urdf.xacro"/>
     <gazebo reference="front_fender_link">
@@ -247,5 +247,5 @@
   </gazebo>
       <gazebo reference="chassis_link">
-    <material>Gazebo/Blue</material>
+    <material>Gazebo/White</material>
   </gazebo>
   <joint name="qrGlue" type="fixed">

Commit message: update

File: jackal_description/urdf/custom_accessories.urdf.xacro (robot description, xacro)
@@ -63,5 +63,5 @@
     <dynamics damping="0.7"/> -->
     <!-- make joint vertical -->
-    <origin rpy="1.5707 0 -1.5707" xyz="0 0 0"/>
+    <origin rpy="1.5707 0 -1.5707" xyz="-0.04 0.0 0.0"/>
     <axis xyz="0 0 1"/>
     <!-- <limit lower="-0.7853982" upper="0.7853982" effort="1000" velocity="10"/>

Commit message: update

File: jackal_description/urdf/custom_accessories.urdf.xacro (robot description, xacro)
@@ -63,6 +63,6 @@
     <dynamics damping="0.7"/> -->
     <!-- make joint vertical -->
-    <origin rpy="1.5707 0 -1.5707" xyz="-0.04 0.0 0.0"/>
-    <axis xyz="0 0 1"/>
+    <origin rpy="1.5707 0 -1.5707" xyz="-0.07 0.0 0.0"/>
+    <axis xyz="0 1 0"/>
     <!-- <limit lower="-0.7853982" upper="0.7853982" effort="1000" velocity="10"/>
     <dynamics damping="0.7"/> -->
@@ -115,5 +115,5 @@
       <inertia
         ixx="1.0" ixy="0.0" ixz="0.0"
-        iyy="1.0" iyz="0.0"
+        iyy="3.0" iyz="0.0"
         izz="1.0"/>
     </inertial>

Commit message: update

File: jackal_description/urdf/custom_accessories.urdf.xacro (robot description, xacro)
@@ -93,9 +93,10 @@
   <link name="custom_tool_link">
     <visual>
-      <!-- <origin xyz="0.3 0 -0.1" rpy="0 -0.7853982 0"/> -->
-      <!-- <origin xyz="0 0 -0.05" rpy="0 0 0"/> -->
       <origin xyz="0 0 -0.075" rpy="0 0 0"/>
-      <geometry>
+      <!-- <geometry>
         <box size="0.005 0.64 0.34"/>
+      </geometry> -->
+        <geometry>
+        <mesh filename="package://smartServoing/models/dozer/dozer.dae" scale="1.0 1.0 1.0"/>
       </geometry>
       <material name="dark_grey" />
@@ -105,7 +106,11 @@
       <!-- <origin xyz="0 0 -0.05" rpy="0 0 0"/> -->
       <origin xyz="0 0 -0.075" rpy="0 0 0"/>
+      <!-- <geometry> -->
+        <!-- <box size="0.005 0.44 0.34"/> -->
+        <!-- <box size="0.005 0.64 0.34"/> -->
+        <!-- <box size="0.005 1.0 0.34"/> -->
+      <!-- </geometry> -->
       <geometry>
-        <!-- <box size="0.005 0.44 0.34"/> -->
-        <box size="0.005 0.64 0.34"/>
+        <mesh filename="package://smartServoing/models/dozer/dozer.dae" scale="1.0 1.0 1.0"/>
       </geometry>
     </collision>
@@ -129,5 +134,5 @@
     </actuator>
   </transmission> -->
-  <gazebo reference="custom_tool_base_link">
+  <!-- <gazebo reference="custom_tool_base_link">
     <material>Gazebo/GreenGlow</material>
     <turnGravityOff>false</turnGravityOff>
@@ -136,5 +141,5 @@
     <material>Gazebo/GreenGlow</material>
     <turnGravityOff>false</turnGravityOff>
-  </gazebo>
+  </gazebo> -->
   <!-- Custom tool model. -->
 </robot>

File: jackal_description/urdf/jackal.urdf.xacro (robot description, xacro)
@@ -34,5 +34,5 @@
       <inertial>
         <origin xyz="0 0 0" rpy="0 0 0"/>
-        <mass value="0.477"/>
+        <mass value="2.0"/>
         <inertia
           ixx="0.0013" ixy="0" ixz="0"
@@ -44,6 +44,6 @@
       <material>Gazebo/DarkGrey</material>
       <selfCollide>false</selfCollide>
-      <mu1 value="0.5"/>
-      <mu2 value="0.5"/>
+      <mu1 value="0.7"/>
+      <mu2 value="0.7"/>
       <kp value="10000000.0" />
       <kd value="1" />
@@ -68,16 +68,4 @@
     </transmission>
   </xacro:macro>
-  <xacro:wheel prefix="front_left">
-    <origin xyz="${wheelbase/2} ${track/2} ${wheel_vertical_offset}" rpy="0 0 0" />
-  </xacro:wheel>
-  <xacro:wheel prefix="front_right">
-    <origin xyz="${wheelbase/2} ${-track/2} ${wheel_vertical_offset}" rpy="0 0 0" />
-  </xacro:wheel>
-  <xacro:wheel prefix="rear_left">
-    <origin xyz="${-wheelbase/2} ${track/2} ${wheel_vertical_offset}" rpy="0 0 0" />
-  </xacro:wheel>
-  <xacro:wheel prefix="rear_right">
-    <origin xyz="${-wheelbase/2} ${-track/2} ${wheel_vertical_offset}" rpy="0 0 0" />
-  </xacro:wheel>
   <link name="base_link"></link>
   <joint name="base_link_joint" type="fixed">
@@ -104,9 +92,9 @@
       <origin xyz="0.012  0.002 0.067" rpy="0 0 0"/>
       <!-- <mass value="16.523"/> -->
-      <mass value="30.000"/>
+      <mass value="50"/>
       <!-- Moments of inertia: ( chassis without wheels ) -->
       <inertia
-        ixx="0.3136" ixy="-0.0008" ixz="0.0164"
-        iyy="0.3922" iyz="-0.0009"
+        ixx="0.3136" ixy="-0.1" ixz="0.1"
+        iyy="0.3922" iyz="-0.1"
         izz="0.4485"/>
       </inertial>
@@ -234,4 +222,16 @@
     <origin xyz="${mount_spacing} 0 0" />
   </joint>
+  <xacro:wheel prefix="front_left">
+    <origin xyz="${wheelbase/2} ${track/2} ${wheel_vertical_offset}" rpy="0 0 0" />
+  </xacro:wheel>
+  <xacro:wheel prefix="front_right">
+    <origin xyz="${wheelbase/2} ${-track/2} ${wheel_vertical_offset}" rpy="0 0 0" />
+  </xacro:wheel>
+  <xacro:wheel prefix="rear_left">
+    <origin xyz="${-wheelbase/2} ${track/2} ${wheel_vertical_offset}" rpy="0 0 0" />
+  </xacro:wheel>
+  <xacro:wheel prefix="rear_right">
+    <origin xyz="${-wheelbase/2} ${-track/2} ${wheel_vertical_offset}" rpy="0 0 0" />
+  </xacro:wheel>
   <!-- Bring in simulation data for Gazebo. -->
   <xacro:include filename="$(find jackal_description)/urdf/jackal.gazebo" />
